File: kicad/ver1.1/snapVCC.sch (KiCad schematic (older format))
At the start: 15 parts, among them P1 CONN_01X03, P2 CONN_01X02, Q1 IRLML9301TRPbF, U1 TPS560200

Commit message: updated schematic
Parts:
- R3: value R -> 20k; Link1 (none) -> Value
Changed lines of the file:
@@
 P 7700 5350
 F 0 "R3" V 7780 5350 50  0000 C CNN
-F 1 "R" V 7700 5350 50  0000 C CNN
+F 1 "20k" V 7700 5350 50  0000 C CNN
 F 2 "" V 7630 5350 30  0000 C CNN
 F 3 "" H 7700 5350 30  0000 C CNN
+F 4 "Value" H 7700 5350 60  0001 C CNN "Link1"
 	1    7700 5350
 	1    0    0    -1
