File: kicad/ver1.1/snapVCC.sch (KiCad schematic (older format))
At the start: 16 parts, among them J1 Jumper Shunt, P1 CONN_01X03, P2 CONN_01X02, Q1 IRLML9301TRPbF, U1 TPS560200

Commit message: fixed 0402 footprint issues
Parts:
- C2: footprint snapVCC_lib:0402-CAP -> snapVCC_lib:0402-seeed
- D1: footprint snapVCC_lib:LED-0603 -> snapVCC_lib:SML-P11_LED_0402
- P1: footprint Connect:PINHEAD1-3 -> snapVCC_lib:PINHEAD1-3
- R4: footprint Resistors_SMD:R_0402 -> snapVCC_lib:0603-RES
- U1: footprint Housings_SOT-23_SOT-143_TSOT-6:SOT-23-5 -> snapVCC_lib:SOT-23-5
Changed lines of the file:
@@
 F 0 "U1" H 5250 3500 60  0000 C CNN
 F 1 "TPS560200" H 5250 4300 60  0000 C CNN
-F 2 "Housings_SOT-23_SOT-143_TSOT-6:SOT-23-5" H 5250 3900 60  0001 C CNN
+F 2 "snapVCC_lib:SOT-23-5" H 5250 3900 60  0001 C CNN
 F 3 "" H 5250 3900 60  0000 C CNN
 F 4 "TPS560200" H 5250 3900 60  0001 C CNN "MFP"
@@
 F 0 "C2" H 4325 4050 50  0000 L CNN
 F 1 "0.1uF" H 4325 3850 50  0000 L CNN
-F 2 "snapVCC_lib:0402-CAP" H 4338 3800 30  0001 C CNN
+F 2 "snapVCC_lib:0402-seeed" H 4338 3800 30  0001 C CNN
 F 3 "" H 4300 3950 60  0000 C CNN
 F 4 "Capacitor, Ceramic, 25V, X7R, 10%" H 4300 3950 60  0001 C CNN "Characteristics"
@@
 F 0 "P1" H 7000 4900 50  0000 C CNN
 F 1 "CONN_01X03" V 7100 4700 50  0001 C CNN
-F 2 "Connect:PINHEAD1-3" H 7000 4700 60  0001 C CNN
+F 2 "snapVCC_lib:PINHEAD1-3" H 7000 4700 60  0001 C CNN
 F 3 "" H 7000 4700 60  0000 C CNN
 F 4 "1.27 mm pitch, male" H 7000 4700 60  0001 C CNN "Characteristics"
@@
 F 0 "R4" V 3580 4700 50  0000 C CNN
 F 1 "7.1k" V 3500 4700 50  0000 C CNN
-F 2 "Resistors_SMD:R_0402" V 3430 4700 30  0001 C CNN
+F 2 "snapVCC_lib:0603-RES" V 3430 4700 30  0001 C CNN
 F 3 "" H 3500 4700 30  0000 C CNN
 F 4 "Resistor, Chip, 1/16W, 1%" H 3500 4700 60  0001 C CNN "Characteristics"
@@
 F 0 "D1" H 3500 4300 50  0000 C CNN
 F 1 "LED" H 3500 4100 50  0000 C CNN
-F 2 "snapVCC_lib:LED-0603" H 3500 4200 60  0001 C CNN
+F 2 "snapVCC_lib:SML-P11_LED_0402" H 3500 4200 60  0001 C CNN
 F 3 "" H 3500 4200 60  0000 C CNN
 F 4 "ROHM" H 3500 4200 60  0001 C CNN "MFN"
