File: kicad/ver1.1/$snapVCC.sch (KiCad schematic (older format))
At the start: 16 parts, among them J1 Jumper Shunt, P1 CONN_01X03, P2 CONN_01X02, Q1 IRLML9301TRPbF, U1 TPS560200

Commit message: done routing
Parts:
- P1: footprint Connect:PINHEAD1-3 -> snapVCC_lib:PINHEAD1-3
- R4: footprint Resistors_SMD:R_0402 -> snapVCC_lib:0603-RES
Changed lines of the file:
@@
 F 0 "P1" H 7000 4900 50  0000 C CNN
 F 1 "CONN_01X03" V 7100 4700 50  0001 C CNN
-F 2 "Connect:PINHEAD1-3" H 7000 4700 60  0001 C CNN
+F 2 "snapVCC_lib:PINHEAD1-3" H 7000 4700 60  0001 C CNN
 F 3 "" H 7000 4700 60  0000 C CNN
 F 4 "1.27 mm pitch, male" H 7000 4700 60  0001 C CNN "Characteristics"
@@
 F 0 "R4" V 3580 4700 50  0000 C CNN
 F 1 "7.1k" V 3500 4700 50  0000 C CNN
-F 2 "Resistors_SMD:R_0402" V 3430 4700 30  0001 C CNN
+F 2 "snapVCC_lib:0603-RES" V 3430 4700 30  0001 C CNN
 F 3 "" H 3500 4700 30  0000 C CNN
 F 4 "Resistor, Chip, 1/16W, 1%" H 3500 4700 60  0001 C CNN "Characteristics"
