File: kicad/ver1.1/snapVCC.kicad_pcb (KiCad board)
At the start: 2 copper layers, 25.9 x 17.3 mm, 17 parts, among them P1 CONN_01X03, P2 CONN_01X02, Q1 IRLML9301TRPbF, U1 TPS560200

Commit message: layout done
Parts:
- moved R1 6.36 mm to (158.2, 105.9)
- moved C3 2.29 mm to (149.4, 101.3)
- moved C2 1.30 mm to (148.6, 109.2)
- moved D1 1.30 mm to (155.4, 101.3)
- moved R4 1.30 mm to (153.2, 102.1)
- moved C4 1.27 mm to (151.1, 101.3)
- moved R3 1.27 mm to (152.1, 109.5)
- moved C1 1.05 mm to (148.6, 110.7)
- moved P1 0.76 mm to (158.0, 110.2)
- moved P2 0.76 mm to (158.2, 100.8)
- moved Q1 0.51 mm to (142.5, 109.5)
- moved G*** 0.36 mm to (138.2, 105.7)
Routing:
- added copper zone on B.Cu, net GND
Other:
- board text added: "+"
- board text added: "-"
- board text added: "3.3V"
- board text added: "5V"
Changed lines of the file:
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@@
   (general
     (links 26)
-    (no_connects 26)
-    (area 135.104572 96.469999 161.594001 113.842001)
+    (no_connects 24)
+    (area 135.585999 96.469999 161.594001 113.842001)
     (thickness 1.6)
-    (drawings 17)
+    (drawings 21)
     (tracks 0)
     (zones 0)
@@
     (last_trace_width 0.25)
     (trace_clearance 0.2)
-    (zone_clearance 0.508)
+    (zone_clearance 0.3)
     (zone_45_only no)
     (trace_min 0.2)
@@
     (add_net "Net-(U1-Pad1)")
   )
+  (module snapVCC_lib:H2-2.54 (layer F.Cu)
+    (at 158.242 100.838)
+    (fp_text reference P2 (at -0.508 -2.794 180) (layer F.SilkS)
+      (effects (font (size 0.4 0.4) (thickness 0.08)) (justify left bottom))
+    )
+    (fp_text value CONN_01X02 (at 1.65 -0.85 90) (layer F.SilkS) hide
+      (effects (font (size 0.4 0.4) (thickness 0.08)) (justify right top))
+    )
+    (pad 1 thru_hole rect (at 0 -1.27) (size 1.651 1.651) (drill 0.889) (layers *.Cu *.Mask)
+      (net 4 "Net-(C3-Pad1)"))
+    (pad 2 thru_hole circle (at 0 1.27) (size 1.651 1.651) (drill 0.889) (layers *.Cu *.Mask)
+      (net 2 GND))
+  )
   (module Housings_SOT-23_SOT-143_TSOT-6:SOT-23-5 (layer F.Cu)
     (at 148.844 106.426 270)
@@
   )
   (module snapVCC_lib:LED-0603 (layer F.Cu)
-    (at 156.718 101.092 270)
-    (fp_text reference D1 (at 0.254 -1.27 450) (layer F.SilkS)
+    (at 155.448 101.346 270)
+    (fp_text reference D1 (at -2.286 -0.254 360) (layer F.SilkS)
       (effects (font (size 0.4 0.4) (thickness 0.08)) (justify right top))
     )
@@
   )
   (module snapVCC_lib:0603-CAP (layer F.Cu)
-    (at 147.574 110.998)
-    (fp_text reference C1 (at -2.25 0.2) (layer F.SilkS)
+    (at 148.59 110.744)
+    (fp_text reference C1 (at -2.54 0.254) (layer F.SilkS)
       (effects (font (size 0.4 0.4) (thickness 0.08)) (justify left bottom))
     )
@@
   )
   (module snapVCC_lib:0402-CAP (layer F.Cu)
-    (at 147.32 109.474)
+    (at 148.59 109.22)
     (descr "<b>CAPACITOR</b><p> chip")
     (attr smd)
-    (fp_text reference C2 (at -1.25 0) (layer F.SilkS)
+    (fp_text reference C2 (at -1.778 0) (layer F.SilkS)
       (effects (font (size 0.4 0.4) (thickness 0.08)) (justify right top))
     )
@@
   )
   (module snapVCC_lib:0603-CAP (layer F.Cu)
-    (at 151.638 101.346 270)
+    (at 149.352 101.346 270)
     (fp_text reference C3 (at -2.032 0.508 540) (layer F.SilkS)
       (effects (font (size 0.4 0.4) (thickness 0.08)) (justify left bottom))
@@
   )
   (module snapVCC_lib:0603-CAP (layer F.Cu)
-    (at 149.86 101.346 270)
-    (fp_text reference C4 (at -2.286 0.508 360) (layer F.SilkS)
+    (at 151.13 101.346 270)
+    (fp_text reference C4 (at -2.032 0.508 360) (layer F.SilkS)
       (effects (font (size 0.4 0.4) (thickness 0.08)) (justify left bottom))
     )
@@
   )
   (module snapVCC_lib:3P-1.27 (layer F.Cu)
-    (at 157.988 109.474 270)
-    (fp_text reference P1 (at -0.95 -0.2 450) (layer F.SilkS)
+    (at 157.988 110.236 270)
+    (fp_text reference P1 (at -0.254 -2.54 540) (layer F.SilkS)
       (effects (font (size 0.4 0.4) (thickness 0.08)) (justify right top))
     )
@@
       (net 8 "Net-(P1-Pad2)"))
   )
-  (module snapVCC_lib:H2-2.54 (layer F.Cu)
-    (at 159.004 100.838)
-    (fp_text reference P2 (at -2.05 0.1 180) (layer F.SilkS)
-      (effects (font (size 0.4 0.4) (thickness 0.08)) (justify left bottom))
-    )
-    (fp_text value CONN_01X02 (at 1.65 -0.85 90) (layer F.SilkS) hide
-      (effects (font (size 0.4 0.4) (thickness 0.08)) (justify right top))
-    )
-    (fp_line (start -1.27 -2.54) (end 1.27 -2.54) (layer F.SilkS) (width 0.127))
-    (fp_line (start 1.27 -2.54) (end 1.27 2.54) (layer F.SilkS) (width 0.127))
-    (fp_line (start 1.27 2.54) (end -1.27 2.54) (layer F.SilkS) (width 0.127))
-    (fp_line (start -1.27 2.54) (end -1.27 -2.54) (layer F.SilkS) (width 0.127))
-    (pad 1 thru_hole rect (at 0 -1.27) (size 1.651 1.651) (drill 0.889) (layers *.Cu *.Mask)
-      (net 4 "Net-(C3-Pad1)"))
-    (pad 2 thru_hole circle (at 0 1.27) (size 1.651 1.651) (drill 0.889) (layers *.Cu *.Mask)
-      (net 2 GND))
-  )
   (module snapVCC_lib:SOT23 (layer F.Cu)
-    (at 142.494 108.966)
+    (at 142.494 109.474)
     (descr <b>SOT23</b>)
     (fp_text reference Q1 (at -2.54 -0.762) (layer F.SilkS)
@@
   )
   (module snapVCC_lib:0603-RES (layer F.Cu)
-    (at 151.892 106.172 270)
-    (fp_text reference R1 (at -1.45 -0.2 270) (layer F.SilkS)
+    (at 158.242 105.918 270)
+    (fp_text reference R1 (at -0.254 -1.778 360) (layer F.SilkS)
       (effects (font (size 0.4 0.4) (thickness 0.08)) (justify right top))
     )
@@
   (module snapVCC_lib:0603-RES (layer F.Cu)
     (at 153.924 109.474 270)
-    (fp_text reference R2 (at -1.45 -0.2 270) (layer F.SilkS)
+    (fp_text reference R2 (at -2.286 -0.254 360) (layer F.SilkS)
       (effects (font (size 0.4 0.4) (thickness 0.08)) (justify right top))
     )
@@
   )
   (module snapVCC_lib:0603-RES (layer F.Cu)
-    (at 150.876 109.474 270)
-    (fp_text reference R3 (at -1.45 -0.2 270) (layer F.SilkS)
+    (at 152.146 109.474 270)
+    (fp_text reference R3 (at -2.286 -0.254 360) (layer F.SilkS)
       (effects (font (size 0.4 0.4) (thickness 0.08)) (justify right top))
     )
@@
   )
   (module Resistors_SMD:R_0402 (layer F.Cu)
-    (at 154.432 101.854 180)
+    (at 153.162 102.108 180)
     (descr "Resistor SMD 0402, reflow soldering, Vishay (see dcrcw.pdf)")
     (tags "resistor 0402")
     (attr smd)
-    (fp_text reference R4 (at -1.778 0 450) (layer F.SilkS)
+    (fp_text reference R4 (at 0 1.27 180) (layer F.SilkS)
       (effects (font (size 0.4 0.4) (thickness 0.1)))
     )
@@
   )
   (module snapVCC_lib:logo-12mm (layer F.Cu)
-    (at 138.43 105.918 90)
+    (at 138.176 105.664 90)
     (fp_text reference G*** (at 0 0 90) (layer F.SilkS) hide
       (effects (font (thickness 0.3)))
@@
       (xy 1.831573 -0.099803) (xy 1.833113 -0.004783) (xy 1.833113 -0.004783)) (layer F.SilkS) (width 0.1))
   )
-  (gr_text electronut.in (at 156.718 112.522) (layer F.SilkS)
+  (gr_text - (at 160.02 102.108) (layer F.SilkS)
+    (effects (font (size 1 1) (thickness 0.2)) (justify mirror))
+  )
+  (gr_text 5V (at 159.004 108.712) (layer F.SilkS)
+    (effects (font (size 0.5 0.5) (thickness 0.1)))
+  )
+  (gr_text 3.3V (at 155.956 108.712) (layer F.SilkS)
+    (effects (font (size 0.5 0.5) (thickness 0.1)))
+  )
+  (gr_text + (at 160.02 99.568) (layer F.SilkS)
+    (effects (font (size 1 1) (thickness 0.2)) (justify mirror))
+  )
+  (gr_text electronut.in (at 156.464 111.76) (layer F.SilkS)
     (effects (font (size 0.8 0.8) (thickness 0.1)))
   )
@@
   (gr_line (start 135.636 98.806) (end 135.636 98.298) (angle 90) (layer Edge.Cuts) (width 0.1))
   (gr_line (start 137.668 96.52) (end 137.16 96.52) (angle 90) (layer Edge.Cuts) (width 0.1))
+  (zone (net 2) (net_name GND) (layer B.Cu) (hatch edge 0.508)
+    (connect_pads (clearance 0.3))
+    (min_thickness 0.0254)
+    (fill yes (arc_segments 16) (thermal_gap 0.3) (thermal_bridge_width 0.4))
+    (polygon
+      (pts
+        (xy 135.636 96.52) (xy 161.544 96.52) (xy 161.544 114.046) (xy 135.636 113.792)
+      )
+    )
+  )
 )

Commit message: updated PCB
Parts:
- P1: footprint snapVCC_lib:3P-1.27 -> PINHEAD1-3
- moved P2 2.81 mm to (158.5, 98.0), turned to 90 degrees
- moved P1 2.17 mm to (157.2, 112.3), turned to 0 degrees
- moved R1 1.83 mm to (159.8, 104.9)
- moved D1 1.78 mm to (157.2, 101.3)
Other:
- board text removed: "-"
Changed lines of the file:
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@@
     (area 135.585999 96.469999 161.594001 113.842001)
     (thickness 1.6)
-    (drawings 21)
+    (drawings 20)
     (tracks 0)
     (zones 0)
@@
     (add_net "Net-(U1-Pad1)")
   )
+  (module PINHEAD1-3 (layer F.Cu)
+    (at 157.226 112.268)
+    (attr virtual)
+    (fp_text reference P1 (at 3.302 -1.524) (layer F.SilkS)
+      (effects (font (size 0.4 0.4) (thickness 0.1)))
+    )
+    (fp_text value CONN_01X03 (at 0 3.81) (layer F.Fab) hide
+      (effects (font (size 1 1) (thickness 0.15)))
+    )
+    (pad 1 thru_hole circle (at -2.54 0) (size 1.65 1.65) (drill 0.889) (layers *.Cu *.Mask)
+      (net 7 "Net-(P1-Pad1)"))
+    (pad 2 thru_hole circle (at 0 0) (size 1.651 1.651) (drill 0.889) (layers *.Cu *.Mask)
+      (net 8 "Net-(P1-Pad2)"))
+    (pad 3 thru_hole circle (at 2.54 0) (size 1.651 1.651) (drill 0.889) (layers *.Cu *.Mask)
+      (net 6 "Net-(P1-Pad3)"))
+  )
   (module snapVCC_lib:H2-2.54 (layer F.Cu)
-    (at 158.242 100.838)
-    (fp_text reference P2 (at -0.508 -2.794 180) (layer F.SilkS)
-      (effects (font (size 0.4 0.4) (thickness 0.08)) (justify left bottom))
-    )
-    (fp_text value CONN_01X02 (at 1.65 -0.85 90) (layer F.SilkS) hide
-      (effects (font (size 0.4 0.4) (thickness 0.08)) (justify right top))
-    )
-    (pad 1 thru_hole rect (at 0 -1.27) (size 1.651 1.651) (drill 0.889) (layers *.Cu *.Mask)
+    (at 158.496 98.044 90)
+    (fp_text reference P2 (at -2.032 -0.254 360) (layer F.SilkS)
+      (effects (font (size 0.4 0.4) (thickness 0.08)) (justify left bottom))
+    )
+    (fp_text value CONN_01X02 (at 1.65 -0.85 180) (layer F.SilkS) hide
+      (effects (font (size 0.4 0.4) (thickness 0.08)) (justify right top))
+    )
+    (pad 1 thru_hole rect (at 0 -1.27 90) (size 1.651 1.651) (drill 0.889) (layers *.Cu *.Mask)
       (net 4 "Net-(C3-Pad1)"))
-    (pad 2 thru_hole circle (at 0 1.27) (size 1.651 1.651) (drill 0.889) (layers *.Cu *.Mask)
+    (pad 2 thru_hole circle (at 0 1.27 90) (size 1.651 1.651) (drill 0.889) (layers *.Cu *.Mask)
       (net 2 GND))
   )
@@
   )
   (module snapVCC_lib:LED-0603 (layer F.Cu)
-    (at 155.448 101.346 270)
+    (at 157.226 101.346 270)
     (fp_text reference D1 (at -2.286 -0.254 360) (layer F.SilkS)
       (effects (font (size 0.4 0.4) (thickness 0.08)) (justify right top))
@@
       (effects (font (size 0.762 0.762) (thickness 0.127)) (justify mirror))
     )
-    (fp_text user [-] (at 6.35 7.366) (layer B.SilkS)
+    (fp_text user [-] (at 6.1849 -7.4676) (layer B.SilkS)
       (effects (font (size 0.762 0.762) (thickness 0.127)) (justify mirror))
     )
@@
     (pad 2 smd rect (at 2 0 90) (size 1.2 3.7) (layers F.Cu F.Paste F.Mask)
       (net 4 "Net-(C3-Pad1)"))
-  )
-  (module snapVCC_lib:3P-1.27 (layer F.Cu)
-    (at 157.988 110.236 270)
-    (fp_text reference P1 (at -0.254 -2.54 540) (layer F.SilkS)
-      (effects (font (size 0.4 0.4) (thickness 0.08)) (justify right top))
-    )
-    (fp_text value CONN_01X03 (at 2.032 -1.27 360) (layer F.SilkS) hide
-      (effects (font (size 0.4 0.4) (thickness 0.08)) (justify right top))
-    )
-    (pad 3 thru_hole circle (at 0 1.905 270) (size 1.016 1.016) (drill 0.635) (layers *.Cu *.Mask)
-      (net 6 "Net-(P1-Pad3)"))
-    (pad 1 thru_hole circle (at 0 -0.635 270) (size 1.016 1.016) (drill 0.635) (layers *.Cu *.Mask)
-      (net 7 "Net-(P1-Pad1)"))
-    (pad 2 thru_hole circle (at 0 0.635 270) (size 1.016 1.016) (drill 0.635) (layers *.Cu *.Mask)
-      (net 8 "Net-(P1-Pad2)"))
   )
   (module snapVCC_lib:SOT23 (layer F.Cu)
@@
   )
   (module snapVCC_lib:0603-RES (layer F.Cu)
-    (at 158.242 105.918 270)
+    (at 159.766 104.902 270)
     (fp_text reference R1 (at -0.254 -1.778 360) (layer F.SilkS)
       (effects (font (size 0.4 0.4) (thickness 0.08)) (justify right top))
@@
       (xy 1.831573 -0.099803) (xy 1.833113 -0.004783) (xy 1.833113 -0.004783)) (layer F.SilkS) (width 0.1))
   )
-  (gr_text - (at 160.02 102.108) (layer F.SilkS)
-    (effects (font (size 1 1) (thickness 0.2)) (justify mirror))
-  )
-  (gr_text 5V (at 159.004 108.712) (layer F.SilkS)
+  (gr_text 5V (at 158.75 110.49) (layer F.SilkS)
     (effects (font (size 0.5 0.5) (thickness 0.1)))
   )
-  (gr_text 3.3V (at 155.956 108.712) (layer F.SilkS)
+  (gr_text 3.3V (at 155.956 110.49) (layer F.SilkS)
     (effects (font (size 0.5 0.5) (thickness 0.1)))
   )
-  (gr_text + (at 160.02 99.568) (layer F.SilkS)
-    (effects (font (size 1 1) (thickness 0.2)) (justify mirror))
-  )
-  (gr_text electronut.in (at 156.464 111.76) (layer F.SilkS)
+  (gr_text + (at 155.194 97.79) (layer F.SilkS)
+    (effects (font (size 1.25 1.25) (thickness 0.2)) (justify mirror))
+  )
+  (gr_text electronut.in (at 148.844 112.522) (layer F.SilkS)
     (effects (font (size 0.8 0.8) (thickness 0.1)))
   )
-  (gr_text "snapVCC 1.1" (at 140.462 98.044) (layer F.SilkS)
+  (gr_text "snapVCC 1.1" (at 148.59 97.79) (layer F.SilkS)
     (effects (font (size 0.8 0.8) (thickness 0.1) italic))
   )

Commit message: updated PCB
Parts:
- added via: VAL**, snapVCC_lib:via, F.Cu at (148.8, 106.4)
- added via: VAL**, snapVCC_lib:via, F.Cu at (140.2, 101.6)
- R1: value 62 -> 62k
- R2: value 43 -> 43k
- moved D1 15.6 mm to (141.7, 99.6), turned to 0 degrees
- moved R4 11.4 mm to (141.7, 101.6)
- moved R3 0.25 mm to (151.9, 109.5)
Connections:
- D1 pad 2: Net-(C3-Pad1) -> Net-(C1-Pad1)
Changed lines of the file:
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@@
 (kicad_pcb (version 4) (host pcbnew "(2015-05-03 BZR 5637)-product")
   (general
-    (links 26)
+    (links 28)
     (no_connects 24)
     (area 134.850572 96.034 162.334334 117.053)
@@
     (tracks 0)
     (zones 0)
-    (modules 17)
+    (modules 19)
     (nets 11)
   )
@@
     (add_net "Net-(U1-Pad1)")
   )
+  (module snapVCC_lib:via (layer F.Cu)
+    (at 148.844 106.426)
+    (fp_text reference via (at 0 -0.508) (layer F.SilkS) hide
+      (effects (font (size 0.4 0.4) (thickness 0.08)))
+    )
+    (fp_text value VAL** (at 0 0.508) (layer F.SilkS) hide
+      (effects (font (size 0.4 0.4) (thickness 0.08)))
+    )
+    (pad 1 thru_hole circle (at 0 0) (size 0.6 0.6) (drill 0.3) (layers *.Cu)
+      (net 2 GND) (zone_connect 2))
+  )
+  (module snapVCC_lib:via (layer F.Cu)
+    (at 140.208 101.6)
+    (fp_text reference via (at 0 -0.508) (layer F.SilkS) hide
+      (effects (font (size 0.4 0.4) (thickness 0.08)))
+    )
+    (fp_text value VAL** (at 0 0.508) (layer F.SilkS) hide
+      (effects (font (size 0.4 0.4) (thickness 0.08)))
+    )
+    (pad 1 thru_hole circle (at 0 0) (size 0.6 0.6) (drill 0.3) (layers *.Cu)
+      (net 2 GND) (zone_connect 2))
+  )
   (module PINHEAD1-3 (layer F.Cu)
     (at 157.226 112.268)
     (attr virtual)
-    (fp_text reference P1 (at 3.302 -1.524) (layer F.SilkS)
-      (effects (font (size 0.4 0.4) (thickness 0.1)))
+    (fp_text reference P1 (at 0.05 -3.8) (layer F.SilkS)
+      (effects (font (size 1 1) (thickness 0.15)))
     )
     (fp_text value CONN_01X03 (at 0 3.81) (layer F.Fab) hide
       (effects (font (size 1 1) (thickness 0.15)))
     )
-    (pad 1 thru_hole circle (at -2.54 0) (size 1.65 1.65) (drill 0.889) (layers *.Cu *.Mask)
+    (pad 1 thru_hole circle (at -2.54 0) (size 1.651 1.651) (drill 0.889) (layers *.Cu *.Mask)
       (net 7 "Net-(P1-Pad1)"))
     (pad 2 thru_hole circle (at 0 0) (size 1.651 1.651) (drill 0.889) (layers *.Cu *.Mask)
@@
   )
   (module snapVCC_lib:LED-0603 (layer F.Cu)
-    (at 157.226 101.346 270)
-    (fp_text reference D1 (at -2.286 -0.254 360) (layer F.SilkS)
-      (effects (font (size 0.4 0.4) (thickness 0.08)) (justify right top))
-    )
-    (fp_text value LED (at 0.762 0.889 270) (layer F.SilkS) hide
+    (at 141.732 99.568)
+    (fp_text reference D1 (at -2.286 -0.254 90) (layer F.SilkS)
+      (effects (font (size 0.4 0.4) (thickness 0.08)) (justify right top))
+    )
+    (fp_text value LED (at 0.762 0.889) (layer F.SilkS) hide
       (effects (font (size 0.4 0.4) (thickness 0.08)) (justify right top))
     )
@@
     (fp_line (start -0.0635 -0.254) (end -0.0635 0.254) (layer F.SilkS) (width 0.127))
     (fp_line (start 0 -0.1905) (end 0 0.1905) (layer F.SilkS) (width 0.127))
-    (pad 2 smd rect (at -0.762 0 270) (size 0.762 0.889) (layers F.Cu F.Paste F.Mask)
-      (net 4 "Net-(C3-Pad1)"))
-    (pad 1 smd rect (at 0.762 0 270) (size 0.762 0.889) (layers F.Cu F.Paste F.Mask)
+    (pad 2 smd rect (at -0.762 0) (size 0.762 0.889) (layers F.Cu F.Paste F.Mask)
+      (net 3 "Net-(C1-Pad1)"))
+    (pad 1 smd rect (at 0.762 0) (size 0.762 0.889) (layers F.Cu F.Paste F.Mask)
       (net 9 "Net-(D1-Pad1)"))
   )
@@
       (effects (font (size 0.762 0.762) (thickness 0.127)) (justify mirror))
     )
-    (fp_text user [-] (at 6.1849 -7.4676) (layer B.SilkS)
-      (effects (font (size 0.762 0.762) (thickness 0.127)) (justify mirror))
-    )
     (pad 1 thru_hole circle (at -6.35 0) (size 3.216 3.216) (drill 2.2) (layers *.Cu *.Mask)
       (net 1 "Net-(BT1-Pad1)"))
@@
       (effects (font (size 0.4 0.4) (thickness 0.08)) (justify right top))
     )
-    (fp_text value 62 (at 0.4 -1.05 270) (layer F.SilkS) hide
+    (fp_text value 62k (at 0.4 -1.05 270) (layer F.SilkS) hide
       (effects (font (size 0.4 0.4) (thickness 0.08)) (justify right top))
     )
@@
       (effects (font (size 0.4 0.4) (thickness 0.08)) (justify right top))
     )
-    (fp_text value 43 (at 0.4 -1.05 270) (layer F.SilkS) hide
+    (fp_text value 43k (at 0.4 -1.05 270) (layer F.SilkS) hide
       (effects (font (size 0.4 0.4) (thickness 0.08)) (justify right top))
     )
@@
   )
   (module snapVCC_lib:0603-RES (layer F.Cu)
-    (at 152.146 109.474 270)
+    (at 151.892 109.474 270)
     (fp_text reference R3 (at -2.286 -0.254 360) (layer F.SilkS)
       (effects (font (size 0.4 0.4) (thickness 0.08)) (justify right top))
@@
   )
   (module Resistors_SMD:R_0402 (layer F.Cu)
-    (at 153.162 102.108 180)
+    (at 141.732 101.6 180)
     (descr "Resistor SMD 0402, reflow soldering, Vishay (see dcrcw.pdf)")
     (tags "resistor 0402")

Commit message: done routing
Parts:
- added via: VAL**, snapVCC_lib:via, F.Cu at (151.6, 112.0)
- added via: VAL**, snapVCC_lib:via, F.Cu at (150.6, 112.0)
- added via: VAL**, snapVCC_lib:via, F.Cu at (140.3, 111.5)
- added via: VAL**, snapVCC_lib:via, F.Cu at (149.6, 112.0)
- added via: VAL**, snapVCC_lib:via, F.Cu at (149.9, 106.4)
- added via: VAL**, snapVCC_lib:via, F.Cu at (147.8, 106.4)
- P1: footprint PINHEAD1-3 -> snapVCC_lib:PINHEAD1-3
- R4: value 3.1k -> 7.1k; footprint Resistors_SMD:R_0402 -> snapVCC_lib:0603-RES
- moved via 0.99 mm to (140.3, 110.5)
- moved via 0.63 mm to (139.6, 101.6)
- moved G*** 0.52 mm to (138.0, 105.2)
Routing:
- net Net-(C1-Pad1): track 0.00 -> 29.8 mm
- net Net-(C3-Pad1): track 0.00 -> 20.3 mm
- net GND: track 0.00 -> 19.5 mm
- net Net-(P1-Pad3): track 0.00 -> 13.9 mm
- net Net-(P1-Pad2): track 0.00 -> 10.3 mm
- net Net-(BT1-Pad1): track 0.00 -> 3.49 mm
- net Net-(D1-Pad1): track 0.00 -> 2.51 mm
- net Net-(L1-Pad1): track 0.00 -> 2.38 mm
- added copper zone on F.Cu, net GND
- added copper zone on F.Cu, net Net-(BT1-Pad1)
- added copper zone on F.Cu, net Net-(C1-Pad1)
- added copper zone on F.Cu, net Net-(C3-Pad1)
- added copper zone on F.Cu, net Net-(L1-Pad1)
Other:
- net class Thick added: clearance 0.2, trace_width 1, via_dia 0.6, via_drill 0.4
- board text added: "3.3"
- board text added: "5"
- board text removed: "3.3V"
- board text removed: "5V"

Commit message: updated U1
Parts:
- U1: footprint Housings_SOT-23_SOT-143_TSOT-6:SOT-23-5 -> SOT-23-5
