File: pcb/ver2.0/snapVCC.sch (KiCad schematic (older format))
At the start: 17 parts, among them J1 Jumper Shunt, P1 CONN_01X03, P2 CONN_01X02, Q1 IRLML9301TRPbF, U1 TPS560200

Commit message: gerbers updated
Parts:
- removed J1: Jumper Shunt, symbol CONN_01X02
Connections:
- no-connect marks 4 -> 2
Changed lines of the file:
@@
 Connection ~ 5700 4400
 Connection ~ 7000 4400
-$Comp
-L CONN_01X02 J1
-U 1 1 56020005
-P 6650 4700
-F 0 "J1" H 6650 4850 50  0000 C CNN
-F 1 "Jumper Shunt" V 6750 4700 50  0000 C CNN
-F 2 "" H 6650 4700 60  0001 C CNN
-F 3 "" H 6650 4700 60  0000 C CNN
-F 4 "Harwin" H 6650 4700 60  0001 C CNN "MFN"
-F 5 "M50-2030005" H 6650 4700 60  0001 C CNN "MFP"
-F 6 "Value" H 6650 4700 60  0001 C CNN "Link1"
-	1    6650 4700
-	-1   0    0    1
-$EndComp
-NoConn ~ 6850 4650
-NoConn ~ 6850 4750
 Wire Wire Line
 	3500 3700 3500 4045

Commit message: gerbers changes updated
Connections:
- net at R1.2, R2.1: now also P1.2 (P2); no longer P1.3 (P3)
Changed lines of the file:
@@
 	1    0    0    -1
 $EndComp
-NoConn ~ 7200 4700
 Connection ~ 3150 5000
 Wire Wire Line
@@
 Wire Wire Line
 	6300 5100 6300 3900
-Connection ~ 7700 4600
-Wire Wire Line
-	7200 4600 7700 4600
 Connection ~ 7700 5100
 Wire Wire Line
@@
 	3500 4840 3500 5000
 Connection ~ 3500 5000
-Wire Wire Line
-	7200 4800 7445 4800
-Wire Wire Line
-	7445 4800 7445 5100
-Connection ~ 7445 5100
 $Comp
 L TEST TP1
@@
 	3500 4445 3500 4540
 Connection ~ 3500 3925
+Wire Wire Line
+	7200 4700 7425 4700
+Wire Wire Line
+	7425 4700 7425 4600
+Wire Wire Line
+	7425 4600 7700 4600
+Connection ~ 7700 4600
+Wire Wire Line
+	7200 4800 7425 4800
+Wire Wire Line
+	7425 4800 7425 5100
+Connection ~ 7425 5100
+NoConn ~ 7200 4600
 $EndSCHEMATC

Commit message: changes updated
Other:
- note added: "3.3V"
Changed lines of the file:
@@
 Connection ~ 7425 5100
 NoConn ~ 7200 4600
+Text Notes 6910 4810 2    60   ~ 0
+3.3V
 $EndSCHEMATC
