File: pcb/ver2.1/snapVCC.kicad_pcb (KiCad board)
At the start: 2 copper layers, 25.9 x 17.3 mm, 26 parts, among them P1 CONN_01X03, P2 CONN_01X02, Q1 IRLML9301TRPbF, U1 TPS560200

Commit message: changes updated
Parts:
- moved G*** 0.51 mm to (137.4, 105.3)
- moved BT1 0.25 mm to (148.1, 105.2)
- moved P1 0.19 mm to (159.2, 107.3)

Commit message: changes updated
Parts:
- moved P2 0.25 mm to (151.0, 99.2)
Other:
- board text added: "snapVCC 2.1"
- board text removed: "snapVCC 2.0"
Changed lines of the file:
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@@
     (links 28)
     (no_connects 2)
-    (area 134.62 96.469999 161.544001 113.842001)
+    (area 135.077999 96.469999 161.086001 113.842001)
     (thickness 0.8)
-    (drawings 25)
+    (drawings 29)
     (tracks 66)
     (zones 0)
@@
   )
   (module snapVCC_lib:H2-2.54 (layer F.Cu)
-    (at 151.257 99.187 180)
+    (at 151.003 99.187 180)
     (fp_text reference P2 (at 1.27 -0.127 180) (layer F.SilkS) hide
       (effects (font (size 0.4 0.4) (thickness 0.08)) (justify left bottom))
@@
       (net 2 GND))
   )
-  (gr_text + (at 149.225 100.33) (layer F.SilkS)
+  (gr_line (start 152.146 99.949) (end 152.908 99.949) (angle 90) (layer F.SilkS) (width 0.1))
+  (gr_line (start 152.146 100.965) (end 152.908 100.965) (angle 90) (layer F.SilkS) (width 0.1))
+  (gr_line (start 152.146 98.425) (end 152.908 98.425) (angle 90) (layer F.SilkS) (width 0.1))
+  (gr_line (start 152.146 97.409) (end 152.908 97.409) (angle 90) (layer F.SilkS) (width 0.1))
+  (gr_text + (at 149.098 100.33) (layer F.SilkS)
     (effects (font (size 1.25 1.25) (thickness 0.2)) (justify mirror))
   )
-  (gr_text - (at 149.352 97.8535 270) (layer F.SilkS)
+  (gr_text - (at 149.225 97.917 270) (layer F.SilkS)
     (effects (font (size 1.5 1.5) (thickness 0.2)))
   )
@@
   (gr_line (start 135.128 112.268) (end 135.128 98.044) (angle 90) (layer Edge.Cuts) (width 0.1))
   (gr_arc (start 158.623 100.457) (end 159.131 99.949) (angle 90) (layer F.SilkS) (width 0.1))
-  (gr_line (start 152.908 99.949) (end 152.908 100.965) (angle 90) (layer F.SilkS) (width 0.1))
-  (gr_line (start 152.908 97.409) (end 152.908 98.425) (angle 90) (layer F.SilkS) (width 0.1))
+  (gr_line (start 152.146 99.949) (end 152.146 100.965) (angle 90) (layer F.SilkS) (width 0.1))
+  (gr_line (start 152.146 97.409) (end 152.146 98.425) (angle 90) (layer F.SilkS) (width 0.1))
   (gr_arc (start 158.623 97.917) (end 159.131 97.409) (angle 90) (layer F.SilkS) (width 0.1))
   (gr_text - (at 160.2105 97.8535 270) (layer F.SilkS)
     (effects (font (size 1.25 1.25) (thickness 0.2)))
   )
-  (gr_text "snapVCC 2.0\n" (at 140.335 97.536) (layer F.SilkS)
+  (gr_text "snapVCC 2.1" (at 140.335 97.536) (layer F.SilkS)
     (effects (font (size 0.8 0.8) (thickness 0.1) italic))
   )
