File: pcb/ver2.1/snapVCC.sch (KiCad schematic (older format))
At the start: 16 parts, among them J1 Jumper Shunt, P1 CONN_01X03, P2 CONN_01X02, Q1 IRLML9301TRPbF, U1 TPS560200

Commit message: ver2.1 updated
Parts:
- removed J1: Jumper Shunt, symbol CONN_01X02
- added TP1: TEST, snapVCC_lib:0R, symbol TEST
- BT1: footprint snapVCC_lib:KEY967 -> snapVCC_lib:KEY967_modified; symbol Battery -> Battery-RESCUE-snapVCC
- C2: footprint snapVCC_lib:0402-seeed -> snapVCC_lib:0603-CAP
- D1: footprint snapVCC_lib:SML-P11_LED_0402 -> LEDs:LED_0603; symbol LED -> LED-RESCUE-snapVCC
- P1: footprint snapVCC_lib:PINHEAD1-3 -> snapVCC_lib:switch
- Q1: symbol Q_PMOS_GSD -> Q_PMOS_GSD-RESCUE-snapVCC
- R4: value 7.1k -> 330R
Connections:
- wire segments 33 -> 35
- no-connect marks 4 -> 2
Other:
- note added: "3.3V"
- moved on the sheet: R4
Changed lines of the file:
@@
 EESchema Schematic File Version 2
+LIBS:snapVCC-rescue
 LIBS:power
 LIBS:device
@@
 Title "snapVCC"
 Date ""
-Rev "1.1"
+Rev "2.0"
 Comp "electronut.in"
 Comment1 ""
@@
 $EndDescr
 $Comp
-L Q_PMOS_GSD Q1
+L Q_PMOS_GSD-RESCUE-snapVCC Q1
 U 1 1 56012F07
 P 3150 3800
-F 0 "Q1" H 3450 3850 50  0000 R CNN
-F 1 "IRLML9301TRPbF" H 3800 3750 50  0000 R CNN
+F 0 "Q1" V 3100 3980 50  0000 R CNN
+F 1 "IRLML9301TRPbF" V 3345 4000 50  0000 R CNN
 F 2 "snapVCC_lib:SOT23" H 3350 3900 29  0001 C CNN
 F 3 "" H 3150 3800 60  0000 C CNN
@@
 $EndComp
 $Comp
-L Battery BT1
+L Battery-RESCUE-snapVCC BT1
 U 1 1 56012F4C
 P 2500 4050
 F 0 "BT1" H 2600 4100 50  0000 L CNN
 F 1 "Battery Holder" H 2600 4000 50  0000 L CNN
-F 2 "snapVCC_lib:KEY967" V 2500 4090 60  0001 C CNN
+F 2 "snapVCC_lib:KEY967_modified" V 2500 4090 60  0001 C CNN
 F 3 "" V 2500 4090 60  0000 C CNN
 F 4 "Keystone" H 2500 4050 60  0001 C CNN "MFN"
@@
 F 0 "C2" H 4325 4050 50  0000 L CNN
 F 1 "0.1uF" H 4325 3850 50  0000 L CNN
-F 2 "snapVCC_lib:0402-seeed" H 4338 3800 30  0001 C CNN
+F 2 "snapVCC_lib:0603-CAP" H 4338 3800 30  0001 C CNN
 F 3 "" H 4300 3950 60  0000 C CNN
 F 4 "Capacitor, Ceramic, 25V, X7R, 10%" H 4300 3950 60  0001 C CNN "Characteristics"
@@
 F 0 "P1" H 7000 4900 50  0000 C CNN
 F 1 "CONN_01X03" V 7100 4700 50  0001 C CNN
-F 2 "snapVCC_lib:PINHEAD1-3" H 7000 4700 60  0001 C CNN
+F 2 "snapVCC_lib:switch" H 7000 4700 60  0001 C CNN
 F 3 "" H 7000 4700 60  0000 C CNN
 F 4 "1.27 mm pitch, male" H 7000 4700 60  0001 C CNN "Characteristics"
@@
 	1    0    0    -1
 $EndComp
-NoConn ~ 7200 4800
 Connection ~ 3150 5000
 Wire Wire Line
@@
 Wire Wire Line
 	8400 3800 8400 4150
-Connection ~ 7500 5100
 Wire Wire Line
 	6300 3900 5700 3900
 Wire Wire Line
 	6300 5100 6300 3900
-Wire Wire Line
-	7500 4700 7500 5100
-Wire Wire Line
-	7200 4700 7500 4700
-Connection ~ 7700 4600
-Wire Wire Line
-	7200 4600 7700 4600
 Connection ~ 7700 5100
 Wire Wire Line
@@
 Connection ~ 3900 3700
 Wire Wire Line
-	3900 3800 3900 3700
+	3900 3700 3900 3800
 Wire Wire Line
 	3350 3700 4800 3700
@@
 L R R4
 U 1 1 56016631
-P 3500 4700
-F 0 "R4" V 3580 4700 50  0000 C CNN
-F 1 "7.1k" V 3500 4700 50  0000 C CNN
-F 2 "snapVCC_lib:0603-RES" V 3430 4700 30  0001 C CNN
-F 3 "" H 3500 4700 30  0000 C CNN
-F 4 "Resistor, Chip, 1/16W, 1%" H 3500 4700 60  0001 C CNN "Characteristics"
-F 5 "0402" H 3500 4700 60  0001 C CNN "Package ID"
-F 6 "Value" H 3500 4700 60  0001 C CNN "Link1"
-	1    3500 4700
-	1    0    0    -1
-$EndComp
-$Comp
-L LED D1
+P 8100 4720
+F 0 "R4" V 8180 4720 50  0000 C CNN
+F 1 "330R" V 8100 4720 50  0000 C CNN
+F 2 "snapVCC_lib:0603-RES" V 8030 4720 30  0001 C CNN
+F 3 "" H 8100 4720 30  0000 C CNN
+F 4 "Resistor, Chip, 1/16W, 1%" H 8100 4720 60  0001 C CNN "Characteristics"
+F 5 "0402" H 8100 4720 60  0001 C CNN "Package ID"
+F 6 "Value" H 8100 4720 60  0001 C CNN "Link1"
+	1    8100 4720
+	1    0    0    -1
+$EndComp
+$Comp
+L LED-RESCUE-snapVCC D1
 U 1 1 56016668
-P 3500 4200
-F 0 "D1" H 3500 4300 50  0000 C CNN
-F 1 "LED" H 3500 4100 50  0000 C CNN
-F 2 "snapVCC_lib:SML-P11_LED_0402" H 3500 4200 60  0001 C CNN
-F 3 "" H 3500 4200 60  0000 C CNN
-F 4 "ROHM" H 3500 4200 60  0001 C CNN "MFN"
-F 5 "SML-P11MT" H 3500 4200 60  0001 C CNN "MFP"
-F 6 "Value" H 3500 4200 60  0001 C CNN "Link1"
-	1    3500 4200
+P 8100 4275
+F 0 "D1" H 8100 4375 50  0000 C CNN
+F 1 "LED" H 8100 4175 50  0000 C CNN
+F 2 "LEDs:LED_0603" H 8100 4275 60  0001 C CNN
+F 3 "" H 8100 4275 60  0000 C CNN
+F 4 "ROHM" H 8100 4275 60  0001 C CNN "MFN"
+F 5 "SML-P11MT" H 8100 4275 60  0001 C CNN "MFP"
+F 6 "Value" H 8100 4275 60  0001 C CNN "Link1"
+	1    8100 4275
 	0    -1   -1   0
 $EndComp
 Connection ~ 5700 4400
 Connection ~ 7000 4400
-$Comp
-L CONN_01X02 J1
-U 1 1 56020005
-P 6650 4700
-F 0 "J1" H 6650 4850 50  0000 C CNN
-F 1 "Jumper Shunt" V 6750 4700 50  0000 C CNN
-F 2 "" H 6650 4700 60  0001 C CNN
-F 3 "" H 6650 4700 60  0000 C CNN
-F 4 "Harwin" H 6650 4700 60  0001 C CNN "MFN"
-F 5 "M50-2030005" H 6650 4700 60  0001 C CNN "MFP"
-F 6 "Value" H 6650 4700 60  0001 C CNN "Link1"
-	1    6650 4700
-	-1   0    0    1
-$EndComp
-NoConn ~ 6850 4650
-NoConn ~ 6850 4750
-Wire Wire Line
-	3500 4000 3500 3700
-Connection ~ 3500 3700
-Wire Wire Line
-	3500 4850 3500 5000
+Wire Wire Line
+	8100 3700 8100 4075
+Wire Wire Line
+	8100 4870 8100 5030
 Connection ~ 3500 5000
-Wire Wire Line
-	3500 4400 3500 4550
+$Comp
+L TEST TP1
+U 1 1 59783D45
+P 8100 3955
+F 0 "TP1" V 8210 4105 50  0000 C BNN
+F 1 "TEST" V 8005 4110 50  0000 C CNN
+F 2 "snapVCC_lib:0R" H 8100 3955 50  0001 C CNN
+F 3 "" H 8100 3955 50  0001 C CNN
+	1    8100 3955
+	0    -1   -1   0
+$EndComp
+Wire Wire Line
+	8100 4475 8100 4570
+Connection ~ 8100 3955
+Wire Wire Line
+	7200 4700 7425 4700
+Wire Wire Line
+	7425 4700 7425 4600
+Wire Wire Line
+	7425 4600 7700 4600
+Connection ~ 7700 4600
+Wire Wire Line
+	7200 4800 7425 4800
+Wire Wire Line
+	7425 4800 7425 5100
+Connection ~ 7425 5100
+NoConn ~ 7200 4600
+Text Notes 6910 4810 2    60   ~ 0
+3.3V
+Connection ~ 8100 3700
+$Comp
+L GND #PWR?
+U 1 1 59897526
+P 8100 5030
+F 0 "#PWR?" H 8100 4780 50  0001 C CNN
+F 1 "GND" H 8100 4880 50  0000 C CNN
+F 2 "" H 8100 5030 60  0000 C CNN
+F 3 "" H 8100 5030 60  0000 C CNN
+	1    8100 5030
+	1    0    0    -1
+$EndComp
 $EndSCHEMATC

Commit message: changes updated
Parts:
- BT1: Link1 Value -> (none); MFN Keystone -> (none); MFP 967 -> (none)
- Q1: Link1 Value -> (none); MFN International Rectifier -> (none); MFP IRLML9301TRPbF -> (none)
- R4: value 330R -> 3K
Other:
- note added: "5V\n"
- moved on the sheet: C1, C2, C3, C4, D1, L1, P1, P2, R1, R2, R3, R4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

Commit message: changes updated
Parts:
- TP1: footprint snapVCC_lib:0R -> (none)
Changed lines of the file:
@@
 $Comp
 L TEST TP1
-U 1 1 598997EE
-P 8280 3140
-F 0 "TP1" H 8280 3355 50  0000 C BNN
-F 1 "TEST" H 8280 3390 50  0001 C CNN
-F 2 "snapVCC_lib:0R" H 8280 3140 50  0001 C CNN
-F 3 "" H 8280 3140 50  0001 C CNN
-	1    8280 3140
+U 1 1 5989908A
+P 8255 3135
+F 0 "TP1" H 8255 3350 50  0000 C BNN
+F 1 "TEST" H 8255 3385 50  0001 C CNN
+F 2 "" H 8255 3135 50  0001 C CNN
+F 3 "" H 8255 3135 50  0001 C CNN
+	1    8255 3135
 	0    -1   -1   0
 $EndComp
 Wire Wire Line
-	8280 3140 8355 3140
-Connection ~ 8355 3140
+	8255 3135 8355 3135
+Connection ~ 8355 3135
 $EndSCHEMATC
